Commit message: Add spot urdf and meshes

File: resources/spot/urdf/spot.urdf (robot description, URDF)
Before this commit: robot spot, 21 links, 20 joints
Links:
- removed link battery
- link base: geometry collision box size=0.7 0.3 0.2; visual mesh filename=package://ocs2_robotic_assets/resources/spot/meshes/base.obj
- link base_inertia: mass 16.0 -> 32.86
Joints:
- removed joint battery_joint
- removed joint body_inertia_joint
- added joint base_inertia_joint: type fixed, parent base, child base_inertia, origin xyz=0 0 0 rpy=0 0 0

Commit message: Update spot's urdf

File: resources/spot/urdf/spot.urdf (robot description, URDF)
Before this commit: robot spot, 20 links, 19 joints
Joints:
- joint LF_HAA: limit lower=-3.14 upper=3.14 effort=1000 velocity=1000.00 -> lower=-0.78539816339744827899 upper=0.78539816339744827899 effort=80 velocity=7.5
- joint LF_HFE: limit lower=-3.14 upper=3.14 effort=1000 velocity=1000.00 -> lower=-0.89884456477707963539 upper=2.2951079663725435509 effort=80 velocity=7.5
- joint LF_KFE: limit lower=-3.14 upper=3.14 effort=1000 velocity=1000.00 -> lower=-2.7929 upper=-0.254402 effort=80 velocity=7.5
- joint LH_HAA: limit lower=-3.14 upper=3.14 effort=1000 velocity=1000.00 -> lower=-0.78539816339744827899 upper=0.78539816339744827899 effort=80 velocity=7.5
- joint LH_HFE: limit lower=-3.14 upper=3.14 effort=1000 velocity=1000.00 -> lower=-0.89884456477707963539 upper=2.2951079663725435509 effort=80 velocity=7.5
- joint LH_KFE: limit lower=-3.14 upper=3.14 effort=1000 velocity=1000.00 -> lower=-2.7929 upper=-0.254402 effort=80 velocity=7.5
- joint RF_HAA: limit lower=-3.14 upper=3.14 effort=1000 velocity=1000.00 -> lower=-0.78539816339744827899 upper=0.78539816339744827899 effort=80 velocity=7.5
- joint RF_HFE: limit lower=-3.14 upper=3.14 effort=1000 velocity=1000.00 -> lower=-0.89884456477707963539 upper=2.2951079663725435509 effort=80 velocity=7.5
- joint RF_KFE: limit lower=-3.14 upper=3.14 effort=1000 velocity=1000.00 -> lower=-2.7929 upper=-0.254402 effort=80 velocity=7.5
- joint RH_HAA: limit lower=-3.14 upper=3.14 effort=1000 velocity=1000.00 -> lower=-0.78539816339744827899 upper=0.78539816339744827899 effort=80 velocity=7.5
- joint RH_HFE: limit lower=-3.14 upper=3.14 effort=1000 velocity=1000.00 -> lower=-0.89884456477707963539 upper=2.2951079663725435509 effort=80 velocity=7.5
- joint RH_KFE: limit lower=-3.14 upper=3.14 effort=1000 velocity=1000.00 -> lower=-2.7929 upper=-0.254402 effort=80 velocity=7.5

Commit message: spotik

File: resources/spot/urdf/spot.urdf (robot description, URDF)
Before this commit: robot spot, 20 links, 19 joints
Links:
- added link camera_link_back, mass 1e-5
- added link camera_link_front_left, mass 1e-5
- added link camera_link_front_right, mass 1e-5
- added link camera_link_left, mass 1e-5
- added link camera_link_right, mass 1e-5
- added link camera_optical_back, mass 1e-5
- added link camera_optical_front_left, mass 1e-5
- added link camera_optical_front_right, mass 1e-5
- added link camera_optical_left, mass 1e-5
- added link camera_optical_right, mass 1e-5
- link base_inertia: mass 32.86 -> 16.0
- link camera_link: mass None -> 1e-5
- link camera_optical: mass None -> 1e-5
- link fl_hip: mass 1.68 -> 2.0
- link fl_lleg: mass 0.35 -> 0.5
- link fl_uleg: mass 2.34 -> 1.0
- link fr_hip: mass 1.68 -> 2.0
- link fr_lleg: mass 0.35 -> 0.5
- link fr_uleg: mass 2.34 -> 1.0
- link hl_hip: mass 1.68 -> 2.0
- link hl_lleg: mass 0.35 -> 0.5
- link hl_uleg: mass 2.34 -> 1.0
- link hr_hip: mass 1.68 -> 2.0
- link hr_lleg: mass 0.35 -> 0.5
- link hr_uleg: mass 2.34 -> 1.0
Joints:
- added joint camera_joint_back: type fixed, parent base, child camera_link_back, origin xyz=-0.425 0 0.01 rpy=0 0.3 -3.141592653589793
- added joint camera_joint_front_left: type fixed, parent base, child camera_link_front_left, origin xyz=0.415 0.037 -0.01 rpy=1.355558 0.353917 -0.554196
- added joint camera_joint_front_right: type fixed, parent base, child camera_link_front_right, origin xyz=0.415 -0.037 -0.01 rpy=-1.355558 0.353917 0.554196
- added joint camera_joint_left: type fixed, parent base, child camera_link_left, origin xyz=-0.125 0.12 0.035 rpy=0 0.2 1.5707963267948966
- added joint camera_joint_right: type fixed, parent base, child camera_link_right, origin xyz=-0.125 -0.12 0.035 rpy=0 0.2 -1.5707963267948966
- added joint camera_optical_joint_back: type fixed, parent camera_link_back, child camera_optical_back, origin xyz=0 0 0 rpy=0 0 0
- added joint camera_optical_joint_front_left: type fixed, parent camera_link_front_left, child camera_optical_front_left, origin xyz=0 0 0 rpy=0 0 0
- added joint camera_optical_joint_front_right: type fixed, parent camera_link_front_right, child camera_optical_front_right, origin xyz=0 0 0 rpy=0 0 0
- added joint camera_optical_joint_left: type fixed, parent camera_link_left, child camera_optical_left, origin xyz=0 0 0 rpy=0 0 0
- added joint camera_optical_joint_right: type fixed, parent camera_link_right, child camera_optical_right, origin xyz=0 0 0 rpy=0 0 0

Commit message: Update visual meshes and collision model

File: resources/spot/urdf/spot.urdf (robot description, URDF)
Before this commit: robot spot, 30 links, 29 joints
Links:
- link base: geometry collision box size=0.7 0.3 0.2; visual mesh filename=package://ocs2_robotic_assets/resources/spot/meshes/visual/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
- link fl_hip: geometry visual mesh filename=package://ocs2_robotic_assets/resources/spot/meshes/visual/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
- link fl_lleg: geometry collision cylinder length=0.30 radius=0.03; collision sphere radius=0.035
- link fl_uleg: geometry collision cylinder length=0.3 radius=0.05; visual mesh filename=package://ocs2_robotic_assets/resources/spot/meshes/visual/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
- link fr_hip: geometry visual mesh filename=package://ocs2_robotic_assets/resources/spot/meshes/visual/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
- link fr_lleg: geometry collision cylinder length=0.30 radius=0.03; collision sphere radius=0.035
- link fr_uleg: geometry collision cylinder length=0.3 radius=0.05; visual mesh filename=package://ocs2_robotic_assets/resources/spot/meshes/visual/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
- link hl_hip: geometry visual mesh filename=package://ocs2_robotic_assets/resources/spot/meshes/visual/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
- link hl_lleg: geometry collision cylinder length=0.30 radius=0.03; collision sphere radius=0.035
- link hl_uleg: geometry collision cylinder length=0.3 radius=0.05; visual mesh filename=package://ocs2_robotic_assets/resources/spot/meshes/visual/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
- link hr_hip: geometry visual mesh filename=package://ocs2_robotic_assets/resources/spot/meshes/visual/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
- link hr_lleg: geometry collision cylinder length=0.30 radius=0.03; collision sphere radius=0.035
- link hr_uleg: geometry collision cylinder length=0.3 radius=0.05; visual mesh filename=package://ocs2_robotic_assets/resources/spot/meshes/visual/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

Commit message: upravene kamery

File: resources/spot/urdf/spot.urdf (robot description, URDF)
Before this commit: robot spot, 30 links, 29 joints
Joints:
- joint camera_joint_left: origin xyz=-0.125 0.12 0.035 rpy=0 0.2 1.5707963267948966 -> xyz=-0.125 0.12 0.035 rpy=3.141592653589793 0.2 1.5707963267948966
- joint camera_joint_right: origin xyz=-0.125 -0.12 0.035 rpy=0 0.2 -1.5707963267948966 -> xyz=-0.125 -0.12 0.035 rpy=3.141592653589793 0.2 -1.5707963267948966
- joint camera_optical_joint_back: origin xyz=0 0 0 rpy=0 0 0 -> xyz=0 0 0 rpy=-1.57 0 -1.57
- joint camera_optical_joint_front_left: origin xyz=0 0 0 rpy=0 0 0 -> xyz=0 0 0 rpy=-1.57 0 -1.57
- joint camera_optical_joint_front_right: origin xyz=0 0 0 rpy=0 0 0 -> xyz=0 0 0 rpy=-1.57 0 -1.57
- joint camera_optical_joint_left: origin xyz=0 0 0 rpy=0 0 0 -> xyz=0 0 0 rpy=-1.57 0 -1.57
- joint camera_optical_joint_right: origin xyz=0 0 0 rpy=0 0 0 -> xyz=0 0 0 rpy=-1.57 0 -1.57
