Commit message: Update description paths

File: resources/anymal_d/urdf/anymal.urdf (robot description, URDF)
Before this commit: robot anymal, 87 links, 86 joints
Links:
- link LF_FOOT: geometry collision cylinder length=0.39572 radius=0.0175; collision sphere radius=0.031455
- link LF_HAA_drive: geometry visual mesh filename=package://ocs2_robotic_assets/resources/anymal_d/meshes/dri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 scale=1.0 1.0 1.0
- link LF_HFE_drive: geometry collision cylinder length=0.119 radius=0.05375; visual mesh filename=package://ocs2_robotic_assets/resources/anymal_d/meshes/dri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 scale=1.0 1.0 1.0
- link LF_KFE_drive: geometry collision cylinder length=0.119 radius=0.05375; visual mesh filename=package://ocs2_robotic_assets/resources/anymal_d/meshes/dri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 scale=1.0 1.0 1.0
- link LF_hip_fixed: geometry visual mesh filename=package://ocs2_robotic_assets/resources/anymal_d/meshes/hip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 scale=1.0 1.0 1.0
- link LF_shank_fixed: geometry collision box size=0.13283 0.08302 0.05732; collision cylinder length=0.05732 radius=0.071
- link LF_thigh_fixed: geometry collision box size=0.093 0.063 0.285; collision cylinder length=0.08313000000000001 radius=0.07
- link LH_FOOT: geometry collision cylinder length=0.39572 radius=0.0175; collision sphere radius=0.031455
- link LH_HAA_drive: geometry visual mesh filename=package://ocs2_robotic_assets/resources/anymal_d/meshes/dri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 scale=1.0 1.0 1.0
- link LH_HFE_drive: geometry collision cylinder length=0.119 radius=0.05375; visual mesh filename=package://ocs2_robotic_assets/resources/anymal_d/meshes/dri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 scale=1.0 1.0 1.0
- link LH_KFE_drive: geometry collision cylinder length=0.119 radius=0.05375; visual mesh filename=package://ocs2_robotic_assets/resources/anymal_d/meshes/dri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 scale=1.0 1.0 1.0
- link LH_hip_fixed: geometry visual mesh filename=package://ocs2_robotic_assets/resources/anymal_d/meshes/hip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 scale=1.0 1.0 1.0
- link LH_shank_fixed: geometry collision box size=0.13283 0.08302 0.05732; collision cylinder length=0.05732 radius=0.071
- link LH_thigh_fixed: geometry collision box size=0.093 0.063 0.285; collision cylinder length=0.08313000000000001 radius=0.07
- link RF_FOOT: geometry collision cylinder length=0.39572 radius=0.0175; collision sphere radius=0.031455
- link RF_HAA_drive: geometry visual mesh filename=package://ocs2_robotic_assets/resources/anymal_d/meshes/dri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 scale=1.0 1.0 1.0
- link RF_HFE_drive: geometry collision cylinder length=0.119 radius=0.05375; visual mesh filename=package://ocs2_robotic_assets/resources/anymal_d/meshes/dri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 scale=1.0 1.0 1.0
- link RF_KFE_drive: geometry collision cylinder length=0.119 radius=0.05375; visual mesh filename=package://ocs2_robotic_assets/resources/anymal_d/meshes/dri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 scale=1.0 1.0 1.0
- link RF_hip_fixed: geometry visual mesh filename=package://ocs2_robotic_assets/resources/anymal_d/meshes/hip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 scale=1.0 1.0 1.0
- link RF_shank_fixed: geometry collision box size=0.13283 0.08302 0.05732; collision cylinder length=0.05732 radius=0.071
- link RF_thigh_fixed: geometry collision box size=0.093 0.063 0.285; collision cylinder length=0.08313000000000001 radius=0.07
- link RH_FOOT: geometry collision cylinder length=0.39572 radius=0.0175; collision sphere radius=0.031455
- link RH_HAA_drive: geometry visual mesh filename=package://ocs2_robotic_assets/resources/anymal_d/meshes/dri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 scale=1.0 1.0 1.0
- link RH_HFE_drive: geometry collision cylinder length=0.119 radius=0.05375; visual mesh filename=package://ocs2_robotic_assets/resources/anymal_d/meshes/dri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 scale=1.0 1.0 1.0
- link RH_KFE_drive: geometry collision cylinder length=0.119 radius=0.05375; visual mesh filename=package://ocs2_robotic_assets/resources/anymal_d/meshes/dri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 scale=1.0 1.0 1.0
- link RH_hip_fixed: geometry visual mesh filename=package://ocs2_robotic_assets/resources/anymal_d/meshes/hip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 scale=1.0 1.0 1.0
- link RH_shank_fixed: geometry collision box size=0.13283 0.08302 0.05732; collision cylinder length=0.05732 radius=0.071
- link RH_thigh_fixed: geometry collision box size=0.093 0.063 0.285; collision cylinder length=0.08313000000000001 radius=0.07
- link base: geometry collision box size=0.894 0.1615 0.256; collision cylinder length=0.1482 radius=0.089
- link battery: geometry visual mesh filename=package://ocs2_robotic_assets/resources/anymal_d/meshes/bat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 scale=1.0 1.0 1.0
- link bottom_shell: geometry visual mesh filename=package://ocs2_robotic_assets/resources/anymal_d/meshes/bot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 scale=1.0 1.0 1.0
- link docking_socket: geometry visual mesh filename=package://ocs2_robotic_assets/resources/anymal_d/meshes/doc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 scale=1.0 1.0 1.0
- link face_shell_front: geometry visual mesh filename=package://ocs2_robotic_assets/resources/anymal_d/meshes/fac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 scale=1.0 1.0 1.0
- link face_shell_rear: geometry visual mesh filename=package://ocs2_robotic_assets/resources/anymal_d/meshes/fac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 scale=1.0 1.0 1.0
- link lidar: geometry collision cylinder length=0.1355 radius=0.07; visual mesh filename=package://ocs2_robotic_assets/resources/anymal_d/meshes/lid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
- link top_shell: geometry visual mesh filename=package://ocs2_robotic_assets/resources/anymal_d/meshes/top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 scale=1.0 1.0 1.0
