Commit message: Rename

File: resources/go2/urdf/go2_description.urdf (robot description, URDF)
Before this commit: robot go2_description, 42 links, 41 joints
Links:
- removed link FL_foot
- removed link FR_foot
- removed link RL_foot
- removed link RR_foot
- added link LF_FOOT, mass 0.04; collision sphere radius=0.022; visual mesh filename=package://ocs2_robotic_assets/resources/go2/dae/foot.dae
- added link LH_FOOT, mass 0.04; collision sphere radius=0.022; visual mesh filename=package://ocs2_robotic_assets/resources/go2/dae/foot.dae
- added link RF_FOOT, mass 0.04; collision sphere radius=0.022; visual mesh filename=package://ocs2_robotic_assets/resources/go2/dae/foot.dae
- added link RH_FOOT, mass 0.04; collision sphere radius=0.022; visual mesh filename=package://ocs2_robotic_assets/resources/go2/dae/foot.dae
Joints:
- removed joint FL_calf_joint
- removed joint FL_foot_joint
- removed joint FL_hip_joint
- removed joint FL_thigh_joint
- removed joint FR_calf_joint
- removed joint FR_foot_joint
- removed joint FR_hip_joint
- removed joint FR_thigh_joint
- removed joint RL_calf_joint
- removed joint RL_foot_joint
- removed joint RL_hip_joint
- removed joint RL_thigh_joint
- removed joint RR_calf_joint
- removed joint RR_foot_joint
- removed joint RR_hip_joint
- removed joint RR_thigh_joint
- added joint LF_FOOT_joint: type fixed, parent FL_calf, child LF_FOOT, origin xyz=0 0 -0.213 rpy=0 0 0, axis 0 0 0
- added joint LF_HAA: type revolute, parent base, child FL_hip, origin xyz=0.1934 0.0465 0 rpy=0 0 0, axis 1 0 0, limit lower=-1.0472 upper=1.0472 effort=23.7 velocity=30.1
- added joint LF_HFE: type revolute, parent FL_hip, child FL_thigh, origin xyz=0 0.0955 0 rpy=0 0 0, axis 0 1 0, limit lower=-1.5708 upper=3.4907 effort=23.7 velocity=30.1
- added joint LF_KFE: type revolute, parent FL_thigh, child FL_calf, origin xyz=0 0 -0.213 rpy=0 0 0, axis 0 1 0, limit lower=-2.7227 upper=-0.83776 effort=45.43 velocity=15.70
- added joint LH_FOOT_joint: type fixed, parent RL_calf, child LH_FOOT, origin xyz=0 0 -0.213 rpy=0 0 0, axis 0 0 0
- added joint LH_HAA: type revolute, parent base, child RL_hip, origin xyz=-0.1934 0.0465 0 rpy=0 0 0, axis 1 0 0, limit lower=-1.0472 upper=1.0472 effort=23.7 velocity=30.1
- added joint LH_HFE: type revolute, parent RL_hip, child RL_thigh, origin xyz=0 0.0955 0 rpy=0 0 0, axis 0 1 0, limit lower=-0.5236 upper=4.5379 effort=23.7 velocity=30.1
- added joint LH_KFE: type revolute, parent RL_thigh, child RL_calf, origin xyz=0 0 -0.213 rpy=0 0 0, axis 0 1 0, limit lower=-2.7227 upper=-0.83776 effort=45.43 velocity=15.70
- added joint RF_FOOT_joint: type fixed, parent FR_calf, child RF_FOOT, origin xyz=0 0 -0.213 rpy=0 0 0, axis 0 0 0
- added joint RF_HAA: type revolute, parent base, child FR_hip, origin xyz=0.1934 -0.0465 0 rpy=0 0 0, axis 1 0 0, limit lower=-1.0472 upper=1.0472 effort=23.7 velocity=30.1
- added joint RF_HFE: type revolute, parent FR_hip, child FR_thigh, origin xyz=0 -0.0955 0 rpy=0 0 0, axis 0 1 0, limit lower=-1.5708 upper=3.4907 effort=23.7 velocity=30.1
- added joint RF_KFE: type revolute, parent FR_thigh, child FR_calf, origin xyz=0 0 -0.213 rpy=0 0 0, axis 0 1 0, limit lower=-2.7227 upper=-0.83776 effort=45.43 velocity=15.70
- added joint RH_FOOT_joint: type fixed, parent RR_calf, child RH_FOOT, origin xyz=0 0 -0.213 rpy=0 0 0, axis 0 0 0
- added joint RH_HAA: type revolute, parent base, child RR_hip, origin xyz=-0.1934 -0.0465 0 rpy=0 0 0, axis 1 0 0, limit lower=-1.0472 upper=1.0472 effort=23.7 velocity=30.1
- added joint RH_HFE: type revolute, parent RR_hip, child RR_thigh, origin xyz=0 -0.0955 0 rpy=0 0 0, axis 0 1 0, limit lower=-0.5236 upper=4.5379 effort=23.7 velocity=30.1
- added joint RH_KFE: type revolute, parent RR_thigh, child RR_calf, origin xyz=0 0 -0.213 rpy=0 0 0, axis 0 1 0, limit lower=-2.7227 upper=-0.83776 effort=45.43 velocity=15.70
